File: hardware/android_debug_cable.kicad_pcb (KiCad board)
At the start: 2 copper layers, 36.7 x 12 mm, 12 parts, among them P1 USB_A, P2 CONN_01X04, P3 SJ-43514-SMT-TR, U1 TPS71718DCKR, U2 CP2103-GM

Commit message: Add v0.2_copperhead
Parts:
- moved W1 1.60 mm to (94.5, 82.1)
- moved C4 0.75 mm to (104.1, 77.8)
- moved C5 0.73 mm to (108.7, 77.9)
- moved U1 0.66 mm to (106.4, 77.9)
Connections:
- P3 pad 2: RX -> TX
- P3 pad 3: TX -> RX
- U1 pad 4: Net-(U1-Pad4) -> (no net)
- U2 pad 1: Net-(U2-Pad1) -> (no net)
- U2 pad 10: Net-(U2-Pad10) -> (no net)
- U2 pad 11: Net-(U2-Pad11) -> (no net)
- U2 pad 12: Net-(U2-Pad12) -> (no net)
- U2 pad 13: Net-(U2-Pad13) -> (no net)
- U2 pad 14: Net-(U2-Pad14) -> (no net)
- U2 pad 15: Net-(U2-Pad15) -> (no net)
- U2 pad 16: Net-(U2-Pad16) -> (no net)
- U2 pad 17: Net-(U2-Pad17) -> (no net)
- U2 pad 18: Net-(U2-Pad18) -> (no net)
- U2 pad 19: Net-(U2-Pad19) -> (no net)
- U2 pad 20: Net-(U2-Pad20) -> (no net)
- U2 pad 21: Net-(U2-Pad21) -> (no net)
- U2 pad 22: Net-(U2-Pad22) -> (no net)
- U2 pad 23: Net-(U2-Pad23) -> (no net)
- U2 pad 26: Net-(U2-Pad26) -> (no net)
- U2 pad 27: Net-(U2-Pad27) -> (no net)
- U2 pad 28: Net-(U2-Pad28) -> (no net)
Routing:
- net RX: track 25.2 -> 42.2 mm, vias 2 -> 3
- net GND: track 63.0 -> 73.6 mm
- net TX: track 23.9 -> 17.1 mm
- net V1.8: track 24.7 -> 25.3 mm
- net Net-(R1-Pad2): track 14.2 -> 14.8 mm
- net VCC: track 56.1 -> 56.6 mm
- removed copper zone on B.Cu, net GND
- removed copper zone on F.Cu, net V3.3
Other:
- board size 36.7 x 12 mm -> 36.7 x 12.2 mm
- board text added: "Android Debug Cable v0.2"
- board text removed: "Android Debug Cable v0.1"
